File: Shield.kicad_pcb (KiCad board)
At the start: 2 copper layers, 54.6 x 53.6 mm, 45 parts, among them J1 Screw_Terminal_01x03, J2 Screw_Terminal_01x03, J3 Screw_Terminal_01x03, J4 Screw_Terminal_01x03, U1 SPX3819M5-L-3-3, U2 SPX3819M5-L-3-3, U3 MAX31865xTP, U4 MAX31865xTP, U5 MAX31865xTP, U6 MAX31865xTP

Commit message: Ajoute img et update connecteur avec 3d
Parts:
- A1: footprint Module:Arduino_UNO_R3 -> Arduino:Arduino_UNO_R3_3d
Changed lines of the file:
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@@
       ))
   )
-  (footprint "Module:Arduino_UNO_R3" (layer "B.Cu")
+  (footprint "Arduino:Arduino_UNO_R3_3d" (layer "B.Cu")
     (at 114.224 90.473)
     (descr "Arduino UNO R3, http://www.mouser.com/pdfdocs/Gravitech_Arduino_Nano3_0.pdf")
@@
     (property "Sheetname" "")
     (attr through_hole)
-    (fp_text reference "A1" (at 1.27 3.81) (layer "B.SilkS")
+    (fp_text reference "A1" (at 1.27 3.81 180) (layer "B.SilkS")
       (effects (font (size 1 1) (thickness 0.15)) (justify mirror))
     )
-    (fp_text value "Arduino_UNO_R3" (at 0 -22.86) (layer "B.Fab") hide
+    (fp_text value "Arduino_UNO_R3" (at 0 -22.86 180) (layer "B.Fab")
       (effects (font (size 1 1) (thickness 0.15)) (justify mirror))
     )
-    (fp_text user "${REFERENCE}" (at -11.1 -16) (layer "B.Fab") hide
+    (fp_text user "${REFERENCE}" (at 0 -20.32 180) (layer "B.Fab")
       (effects (font (size 1 1) (thickness 0.15)) (justify mirror))
     )
+    (fp_line (start -28.07 -41.4) (end -28.07 -50.93) (layer "B.SilkS") (width 0.12))
+    (fp_line (start -28.07 -0.51) (end -29.97 -0.51) (layer "B.SilkS") (width 0.12))
+    (fp_line (start 38.23 0) (end 38.23 2.67) (layer "B.SilkS") (width 0.12))
+    (fp_line (start -34.42 -41.4) (end -28.07 -41.4) (layer "B.SilkS") (width 0.12))
+    (fp_line (start -28.07 -29.72) (end -34.42 -29.72) (layer "B.SilkS") (width 0.12))
+    (fp_line (start -34.42 -29.72) (end -34.42 -41.4) (layer "B.SilkS") (width 0.12))
+    (fp_line (start 40.77 -35.31) (end 40.77 -2.54) (layer "B.SilkS") (width 0.12))
+    (fp_line (start 36.58 -50.93) (end 38.23 -49.28) (layer "B.SilkS") (width 0.12))
+    (fp_line (start 38.23 2.67) (end -28.07 2.67) (layer "B.SilkS") (width 0.12))
+    (fp_line (start -28.07 -9.65) (end -28.07 -29.72) (layer "B.SilkS") (width 0.12))
+    (fp_line (start 38.23 -49.28) (end 38.23 -37.85) (layer "B.SilkS") (width 0.12))
+    (fp_line (start 40.77 -2.54) (end 38.23 0) (layer "B.SilkS") (width 0.12))
+    (fp_line (start -28.07 2.67) (end -28.07 -0.51) (layer "B.SilkS") (width 0.12))
+    (fp_line (start 38.23 -37.85) (end 40.77 -35.31) (layer "B.SilkS") (width 0.12))
+    (fp_line (start -28.07 -50.93) (end 36.58 -50.93) (layer "B.SilkS") (width 0.12))
+    (fp_line (start -29.97 -0.51) (end -29.97 -9.65) (layer "B.SilkS") (width 0.12))
+    (fp_line (start -29.97 -9.65) (end -28.07 -9.65) (layer "B.SilkS") (width 0.12))
+    (fp_line (start -28.19 2.79) (end 38.35 2.79) (layer "B.CrtYd") (width 0.05))
+    (fp_line (start -28.19 -51.05) (end -28.19 -41.53) (layer "B.CrtYd") (width 0.05))
+    (fp_line (start -28.19 -41.53) (end -34.54 -41.53) (layer "B.CrtYd") (width 0.05))
+    (fp_line (start -34.54 -29.59) (end -28.19 -29.59) (layer "B.CrtYd") (width 0.05))
+    (fp_line (start -28.19 -29.59) (end -28.19 -9.78) (layer "B.CrtYd") (width 0.05))
+    (fp_line (start 38.35 0) (end 40.89 -2.54) (layer "B.CrtYd") (width 0.05))
+    (fp_line (start -28.19 -9.78) (end -30.1 -9.78) (layer "B.CrtYd") (width 0.05))
+    (fp_line (start 38.35 -49.28) (end 36.58 -51.05) (layer "B.CrtYd") (width 0.05))
+    (fp_line (start -34.54 -41.53) (end -34.54 -29.59) (layer "B.CrtYd") (width 0.05))
+    (fp_line (start 36.58 -51.05) (end -28.19 -51.05) (layer "B.CrtYd") (width 0.05))
+    (fp_line (start 40.89 -2.54) (end 40.89 -35.31) (layer "B.CrtYd") (width 0.05))
+    (fp_line (start -30.1 -9.78) (end -30.1 -0.38) (layer "B.CrtYd") (width 0.05))
+    (fp_line (start 40.89 -35.31) (end 38.35 -37.85) (layer "B.CrtYd") (width 0.05))
+    (fp_line (start 38.35 2.79) (end 38.35 0) (layer "B.CrtYd") (width 0.05))
+    (fp_line (start -28.19 -0.38) (end -28.19 2.79) (layer "B.CrtYd") (width 0.05))
+    (fp_line (start -30.1 -0.38) (end -28.19 -0.38) (layer "B.CrtYd") (width 0.05))
+    (fp_line (start 38.35 -37.85) (end 38.35 -49.28) (layer "B.CrtYd") (width 0.05))
+    (fp_line (start -29.84 -0.64) (end -16.51 -0.64) (layer "B.Fab") (width 0.1))
+    (fp_line (start -34.29 -41.27) (end -34.29 -29.84) (layer "B.Fab") (width 0.1))
+    (fp_line (start 40.64 -2.54) (end 40.64 -35.31) (layer "B.Fab") (width 0.1))
+    (fp_line (start -27.94 -50.8) (end -27.94 2.54) (layer "B.Fab") (width 0.1))
+    (fp_line (start -18.41 -29.84) (end -18.41 -41.27) (layer "B.Fab") (width 0.1))
+    (fp_line (start 38.1 -49.28) (end 36.58 -50.8) (layer "B.Fab") (width 0.1))
+    (fp_line (start -27.94 2.54) (end 38.1 2.54) (layer "B.Fab") (width 0.1))
+    (fp_line (start 36.58 -50.8) (end -27.94 -50.8) (layer "B.Fab") (width 0.1))
+    (fp_line (start -34.29 -29.84) (end -18.41 -29.84) (layer "B.Fab") (width 0.1))
+    (fp_line (start 40.64 -35.31) (end 38.1 -37.85) (layer "B.Fab") (width 0.1))
+    (fp_line (start -18.41 -41.27) (end -34.29 -41.27) (layer "B.Fab") (width 0.1))
+    (fp_line (start -16.51 -0.64) (end -16.51 -9.53) (layer "B.Fab") (width 0.1))
+    (fp_line (start 38.1 2.54) (end 38.1 0) (layer "B.Fab") (width 0.1))
+    (fp_line (start -16.51 -9.53) (end -29.84 -9.53) (layer "B.Fab") (width 0.1))
+    (fp_line (start 38.1 -37.85) (end 38.1 -49.28) (layer "B.Fab") (width 0.1))
+    (fp_line (start 38.1 0) (end 40.64 -2.54) (layer "B.Fab") (width 0.1))
+    (fp_line (start -29.84 -9.53) (end -29.84 -0.64) (layer "B.Fab") (width 0.1))
     (pad "1" thru_hole rect (at 0 0 270) (size 1.6 1.6) (drill 1) (layers *.Cu *.Mask)
       (net 38 "unconnected-(A1-Pad1)") (pinfunction "NC") (pintype "no_connect"))
@@
     (pad "32" thru_hole oval (at -9.14 -48.26 270) (size 1.6 1.6) (drill 1) (layers *.Cu *.Mask)
       (net 63 "unconnected-(A1-Pad32)") (pinfunction "SCL/A5") (pintype "bidirectional+no_connect"))
-    (model "${KICAD6_3DMODEL_DIR}/Connector_PinHeader_2.54mm.3dshapes/PinHeader_1x11_P2.54mm_Vertical.wrl" hide
+    (model "${KICAD6_3DMODEL_DIR}/Module.3dshapes/Arduino_UNO_R3.wrl"
       (offset (xyz 0 0 0))
       (scale (xyz 1 1 1))
       (rotate (xyz 0 0 0))
     )
+    (model "/home/gaby/GitRepo/3d_conn_misc/walter/conn_misc.3dshapes/arduino_header.wrl"
+      (offset (xyz 5 -24 -1.5))
+      (scale (xyz 1 1 1))
+      (rotate (xyz 0 -180 -180))
+    )
   )

Commit message: Ajoute selection 4w/3w Ajoute marquage v002
Parts:
- added JP13: SolderJumper_3_Open, Jumper:SolderJumper-3_P1.3mm_Open_RoundedPad1.0x1.5mm_NumberLabels, B.Cu at (147.4, 85.4)
- added JP14: SolderJumper_3_Open, Jumper:SolderJumper-3_P1.3mm_Open_RoundedPad1.0x1.5mm_NumberLabels, B.Cu at (147.3, 80.4)
- added JP15: SolderJumper_3_Open, Jumper:SolderJumper-3_P1.3mm_Open_RoundedPad1.0x1.5mm_NumberLabels, B.Cu at (147.3, 74.3)
- added JP16: SolderJumper_3_Open, Jumper:SolderJumper-3_P1.3mm_Open_RoundedPad1.0x1.5mm_NumberLabels, B.Cu at (147.4, 69.3)
- added JP17: SolderJumper_3_Open, Jumper:SolderJumper-3_P1.3mm_Open_RoundedPad1.0x1.5mm_NumberLabels, B.Cu at (147.4, 63.3)
- added JP18: SolderJumper_3_Open, Jumper:SolderJumper-3_P1.3mm_Open_RoundedPad1.0x1.5mm_NumberLabels, B.Cu at (147.3, 58.2)
- added JP19: SolderJumper_3_Open, Jumper:SolderJumper-3_P1.3mm_Open_RoundedPad1.0x1.5mm_NumberLabels, B.Cu at (147.2, 52.9)
- added JP20: SolderJumper_3_Open, Jumper:SolderJumper-3_P1.3mm_Open_RoundedPad1.0x1.5mm_NumberLabels, B.Cu at (147.2, 47.1)
- J1, J2, J3, J4: value Screw_Terminal_01x03 -> Screw_Terminal_01x04; footprint TerminalBlock_Phoenix:TerminalBlock_Phoenix_MPT-0,5-3-2.54_1x03_P2.54mm_Horizontal -> TerminalBlock_Phoenix:TerminalBlock_Phoenix_MPT-0,5-4-2.54_1x04_P2.54mm_Horizontal
- moved J4 3.70 mm to (152.1, 52.9)
- moved J1 3.64 mm to (152.1, 87.0)
- moved J3 3.20 mm to (152.1, 64.2)
- moved J2 3.12 mm to (152.1, 75.6)
Connections:
- U3 pad 6: Net-(J1-Pad1) -> Net-(JP13-Pad2)
- U3 pad 9: Net-(C10-Pad1) -> Net-(JP14-Pad2)
- U4 pad 6: Net-(J2-Pad1) -> Net-(JP15-Pad2)
- U4 pad 9: Net-(C12-Pad1) -> Net-(JP16-Pad2)
- U5 pad 6: Net-(J3-Pad1) -> Net-(JP17-Pad2)
- U5 pad 9: Net-(C15-Pad1) -> Net-(JP18-Pad2)
- U6 pad 6: Net-(J4-Pad1) -> Net-(JP19-Pad2)
- U6 pad 9: Net-(C18-Pad1) -> Net-(JP20-Pad2)
Routing:
- net Net-(JP14-Pad2): track 0.00 -> 8.84 mm, vias 0 -> 1
- net Net-(JP16-Pad2): track 0.00 -> 8.06 mm, vias 0 -> 1
- net Net-(JP20-Pad2): track 0.00 -> 7.50 mm, vias 0 -> 1
- net Net-(JP18-Pad2): track 0.00 -> 7.29 mm, vias 0 -> 1
- net Net-(JP13-Pad2): track 0.00 -> 6.63 mm, vias 0 -> 1
- net Net-(JP15-Pad2): track 0.00 -> 6.14 mm, vias 0 -> 1
- net Net-(JP17-Pad2): track 0.00 -> 5.78 mm, vias 0 -> 1
- net Net-(JP19-Pad2): track 0.00 -> 5.76 mm, vias 0 -> 1
- net Net-(J4-Pad4): track 0.00 -> 5.06 mm
- net Net-(J3-Pad4): track 0.00 -> 4.93 mm
- net Net-(J1-Pad4): track 0.00 -> 4.87 mm
- net Net-(J2-Pad4): track 0.00 -> 4.71 mm
- net Net-(C10-Pad2): track 8.08 -> 12.0 mm, vias 0 -> 1
- net Net-(C10-Pad1): track 10.1 -> 13.5 mm, vias 0 -> 1
- net Net-(C12-Pad2): track 8.08 -> 11.4 mm, vias 0 -> 1
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Other:
- board size 54.6 x 53.6 mm -> 52.5 x 53.6 mm
- board text added: "3V3"
- board text added: "3w 3 2+ 1+ 3 2+ 1+"
- board text added: "4w 3+ 2+ 1 3+ 2+ 1"
- board text added: "5V"
- board text added: "A0/CS1"
- board text added: "A1/CS2"
- board text added: "A2/CS3"
- board text added: "A3/CS4"
- board text added: "A4"
- board text added: "A5"
- board text added: "AVDD"
- board text added: "D0"
- board text added: "D1"
- board text added: "D10"
- board text added: "D11/SPI MOSI"
- board text added: "D12/SPI MISO"
- board text added: "D13/SCK"
- board text added: "D14"
- board text added: "D15"
- board text added: "D2/CS1"
- board text added: "D3/CS2"
- board text added: "D4/CS3"
- board text added: "D5/CS4"
- board text added: "D6/CS1"
- board text added: "D7/CS2"
- board text added: "D8/CS3"
- board text added: "D9/CS4"
- board text added: "GND"
- board text added: "IOREF"
- board text added: "NRST"
- board text added: "VIN"
